Commit message: fix: place body above wheels

File: urdf/ackermann_robot.urdf.xacro (robot description, xacro)
@@ -12,5 +12,6 @@
   <xacro:property name="body_width" value="0.300"/>
   <xacro:property name="body_height" value="0.165"/>
-  <xacro:property name="ground_clearance" value="0.030"/>
+  <!-- Place the main body above the tires; wheel top is 2 * wheel_radius. -->
+  <xacro:property name="body_bottom_z" value="${2.0 * wheel_radius}"/>
   <!-- Measured running gear. -->
   <xacro:property name="wheelbase" value="0.2775"/>
@@ -24,5 +25,5 @@
                   value="${(body_rear_x + body_front_x) / 2.0}"/>
   <xacro:property name="body_center_z"
-                  value="${ground_clearance + body_height / 2.0}"/>
+                  value="${body_bottom_z + body_height / 2.0}"/>
   <!-- Sensor centers measured from base_link. -->
   <xacro:property name="lidar_x" value="0.237"/>

Commit message: fix: size chassis between wheel centers

File: urdf/ackermann_robot.urdf.xacro (robot description, xacro)
@@ -8,10 +8,4 @@
     joints because the robot has no wheel position or steering encoders.
   -->
-  <!-- Measured body geometry. -->
-  <xacro:property name="body_length" value="0.385"/>
-  <xacro:property name="body_width" value="0.300"/>
-  <xacro:property name="body_height" value="0.165"/>
-  <!-- Place the main body above the tires; wheel top is 2 * wheel_radius. -->
-  <xacro:property name="body_bottom_z" value="${2.0 * wheel_radius}"/>
   <!-- Measured running gear. -->
   <xacro:property name="wheelbase" value="0.2775"/>
@@ -19,11 +13,10 @@
   <xacro:property name="wheel_radius" value="0.060"/>
   <xacro:property name="wheel_width" value="0.057"/>
-  <!-- Body extents relative to the rear axle. -->
-  <xacro:property name="body_rear_x" value="-0.0538"/>
-  <xacro:property name="body_front_x" value="0.3312"/>
-  <xacro:property name="body_center_x"
-                  value="${(body_rear_x + body_front_x) / 2.0}"/>
-  <xacro:property name="body_center_z"
-                  value="${body_bottom_z + body_height / 2.0}"/>
+  <!-- Thin chassis plate: axle-to-axle and between the inner tire faces. -->
+  <xacro:property name="body_length" value="${wheelbase}"/>
+  <xacro:property name="body_width" value="${track_width - wheel_width}"/>
+  <xacro:property name="body_height" value="${wheel_radius}"/>
+  <xacro:property name="body_center_x" value="${wheelbase / 2.0}"/>
+  <xacro:property name="body_center_z" value="${1.5 * wheel_radius}"/>
   <!-- Sensor centers measured from base_link. -->
   <xacro:property name="lidar_x" value="0.237"/>

Commit message: fix: use measured chassis length

File: urdf/ackermann_robot.urdf.xacro (robot description, xacro)
@@ -13,9 +13,12 @@
   <xacro:property name="wheel_radius" value="0.060"/>
   <xacro:property name="wheel_width" value="0.057"/>
-  <!-- Thin chassis plate: axle-to-axle and between the inner tire faces. -->
-  <xacro:property name="body_length" value="${wheelbase}"/>
+  <!-- Thin chassis plate: measured body length, between inner tire faces. -->
+  <xacro:property name="body_rear_x" value="-0.0538"/>
+  <xacro:property name="body_front_x" value="0.3312"/>
+  <xacro:property name="body_length" value="${body_front_x - body_rear_x}"/>
   <xacro:property name="body_width" value="${track_width - wheel_width}"/>
   <xacro:property name="body_height" value="${wheel_radius}"/>
-  <xacro:property name="body_center_x" value="${wheelbase / 2.0}"/>
+  <xacro:property name="body_center_x"
+                  value="${(body_front_x + body_rear_x) / 2.0}"/>
   <xacro:property name="body_center_z" value="${1.5 * wheel_radius}"/>
   <!-- Sensor centers measured from base_link. -->
